File: keyboard-pcb-tutorial.kicad_pcb (KiCad board)
At the start: 2 copper layers, 93.7 x 38.1 mm, 24 parts, among them SW1 SW_Push, U1 ATmega32U4-AU, Y1 16MHz

Commit message: Fill zones, decoration and production
Routing:
- net GND: track 142.9 -> 140.5 mm
- added copper zone on B.Cu, net GND
Other:
- board text added: "GreatWizard — 2020 —"
Changed lines of the file:
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@@
   (general
     (thickness 1.6)
-    (drawings 8)
-    (tracks 197)
+    (drawings 9)
+    (tracks 194)
     (zones 0)
     (modules 24)
@@
     (visible_elements FFFFFF7F)
     (pcbplotparams
-      (layerselection 0x010fc_ffffffff)
+      (layerselection 0x010f0_ffffffff)
       (usegerberextensions false)
       (usegerberattributes false)
@@
       (outputformat 1)
       (mirror false)
-      (drillshape 1)
+      (drillshape 0)
       (scaleselection 1)
-      (outputdirectory ""))
+      (outputdirectory "Gerbers"))
   )
   (net 0 "")
@@
     )
   )
+  (gr_text "GreatWizard\n— 2020 — " (at 161.13125 159.54375) (layer F.SilkS)
+    (effects (font (size 1 1) (thickness 0.15)))
+  )
   (gr_line (start 134.9375 129.38125) (end 134.9375 162.71875) (layer Edge.Cuts) (width 0.05))
   (gr_line (start 226.21875 127) (end 137.31875 127) (layer Edge.Cuts) (width 0.05))
@@
   (segment (start 171.425 153.21875) (end 171.425 151.75) (width 0.381) (layer B.Cu) (net 1))
   (segment (start 170.65625 153.9875) (end 171.425 153.21875) (width 0.381) (layer B.Cu) (net 1))
-  (segment (start 169.71875 135.5875) (end 169.71875 134.14375) (width 0.381) (layer B.Cu) (net 1))
-  (segment (start 163.5125 135.5875) (end 169.71875 135.5875) (width 0.381) (layer B.Cu) (net 1))
-  (segment (start 169.71875 134.14375) (end 169.06875 133.49375) (width 0.381) (layer B.Cu) (net 1))
-  (segment (start 169.71875 135.5875) (end 172.89375 135.5875) (width 0.381) (layer B.Cu) (net 1))
+  (segment (start 163.5125 135.5875) (end 172.89375 135.5875) (width 0.381) (layer B.Cu) (net 1))
   (segment (start 174.625 133.7125) (end 174.93125 133.40625) (width 0.254) (layer B.Cu) (net 2))
   (segment (start 174.625 140.35) (end 174.625 133.7125) (width 0.254) (layer B.Cu) (net 2))
@@
   (segment (start 171.704249 134.267851) (end 171.911949 134.475551) (width 0.254) (layer B.Cu) (net 3))
   (segment (start 171.911949 134.475551) (end 172.506388 135.06999) (width 0.254) (layer B.Cu) (net 3))
-  (segment (start 172.3 131.70625) (end 172.73125 131.70625) (width 0.254) (layer B.Cu) (net 3))
-  (segment (start 171.45 132.55625) (end 172.3 131.70625) (width 0.254) (layer B.Cu) (net 3))
-  (segment (start 171.45 134.013602) (end 171.45 132.55625) (width 0.254) (layer B.Cu) (net 3))
+  (segment (start 171.77725 131.70625) (end 172.73125 131.70625) (width 0.254) (layer B.Cu) (net 3))
+  (segment (start 171.45 132.0335) (end 171.77725 131.70625) (width 0.254) (layer B.Cu) (net 3))
+  (segment (start 171.45 134.013602) (end 171.45 132.0335) (width 0.254) (layer B.Cu) (net 3))
   (segment (start 171.911949 134.475551) (end 171.45 134.013602) (width 0.254) (layer B.Cu) (net 3))
   (segment (start 172.225 138.38125) (end 172.225 140.35) (width 0.381) (layer B.Cu) (net 5))
@@
   (segment (start 182.70625 149.875) (end 182.53125 150.05) (width 0.254) (layer B.Cu) (net 20))
   (segment (start 184.15 149.875) (end 182.70625 149.875) (width 0.254) (layer B.Cu) (net 20))
+  (zone (net 1) (net_name GND) (layer B.Cu) (hatch edge 0.508)
+    (connect_pads (clearance 0.508))
+    (min_thickness 0.254)
+    (fill yes (arc_segments 32) (thermal_gap 0.508) (thermal_bridge_width 0.508))
+    (polygon
+      (pts
+        (xy 134.9375 127) (xy 190.5 127) (xy 190.5 165.1) (xy 134.9375 165.1)
+      )
+    )
+  )
 )
